File: elec/layouts/debug/servo-drive.kicad_pcb (KiCad board)
At the start: 4 copper layers, 85.3 x 55.9 mm, 84 parts

Commit message: lots of dumb little mistaktes
Parts:
- C10, C11, C12, C13, C14, C9: footprint Capacitor_SMD:C_0603_1608Metric -> Capacitor_SMD:C_0402_1005Metric
- R1, R11, R12, R13, R14, R15, R16, R17, R18, R19, R2, R20, R21, R22, R23, R24, R25, R26, R27, R28, R29, R3, R30, R5, R6, R8, R9: footprint Resistor_SMD:R_0603_1608Metric -> Resistor_SMD:R_0402_1005Metric
